File: pcb/cornechon.kicad_sch (KiCad schematic)
At the start: 69 parts, among them J1 MJ-4PP-9, J2 Conn_01x04, J3 Conn_01x02_Female, K1 KEYSW, K10 KEYSW, K11 KEYSW, K12 KEYSW, K13 KEYSW, K14 KEYSW, K15 KEYSW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

Commit message: add kb info
Other:
- title: Nijuni -> Cornechon
